Commit message: グローサ形状を円形に変更:シミュレーション時の接触状態が安定化する

File: urdf/default_crawler.urdf (robot description, URDF)
Before this commit: robot crawler, 24 links, 23 joints
Links:
- link flipper_idler_left_front: geometry collision cylinder length=0.025 radius=0.112; visual cylinder length=0.025 radius=0.082
- link flipper_idler_left_rear: geometry collision cylinder length=0.025 radius=0.112; visual cylinder length=0.025 radius=0.082
- link flipper_idler_right_front: geometry collision cylinder length=0.025 radius=0.112; visual cylinder length=0.025 radius=0.082
- link flipper_idler_right_rear: geometry collision cylinder length=0.025 radius=0.112; visual cylinder length=0.025 radius=0.082
- link flipper_sprocket_left_front: geometry collision cylinder length=0.025 radius=0.112; visual cylinder length=0.025 radius=0.082
- link flipper_sprocket_left_rear: geometry collision cylinder length=0.025 radius=0.112; visual cylinder length=0.025 radius=0.082
- link flipper_sprocket_right_front: geometry collision cylinder length=0.025 radius=0.112; visual cylinder length=0.025 radius=0.082
- link flipper_sprocket_right_rear: geometry collision cylinder length=0.025 radius=0.112; visual cylinder length=0.025 radius=0.082
- link idler_left: geometry collision cylinder length=0.1 radius=0.112; visual cylinder length=0.1 radius=0.082
- link idler_right: geometry collision cylinder length=0.1 radius=0.112; visual cylinder length=0.1 radius=0.082
- link sprocket_left: geometry collision cylinder length=0.1 radius=0.112; visual cylinder length=0.1 radius=0.082
- link sprocket_right: geometry collision cylinder length=0.1 radius=0.112; visual cylinder length=0.1 radius=0.082
Joints:
- joint joint_left_front: limit lower=-2.35619449 upper=2.35619449 effort=8000 velocity=1 -> lower=-2.35619449 upper=2.35619449 effort=20000 velocity=10
- joint joint_left_rear: limit lower=-2.35619449 upper=2.35619449 effort=8000 velocity=1 -> lower=-2.35619449 upper=2.35619449 effort=20000 velocity=10
- joint joint_right_front: limit lower=-2.35619449 upper=2.35619449 effort=8000 velocity=1 -> lower=-2.35619449 upper=2.35619449 effort=20000 velocity=10
- joint joint_right_rear: limit lower=-2.35619449 upper=2.35619449 effort=8000 velocity=1 -> lower=-2.35619449 upper=2.35619449 effort=20000 velocity=10
